File: line_sensor_color/line_sensor_color.sch (KiCad schematic (older format))
At the start: 59 parts, among them SW1 SW_DIP_x03, SW2 SW_DIP_x03, SW3 SW_DIP_x03, SW4 SW_DIP_x03, SW5 SW_DIP_x03, SW6 SW_DIP_x03, U1 XH_2, U2 XH_2, U3 XH_2, U4 NJM7800SDL1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

Commit message: update: フットプリントに3Dデータを追加
Parts:
- A1: footprint MODULE_NUCLEO-F303K8 -> MyFootprint:NUCLEO_F303K8
Changed lines of the file:
@@
 EESchema Schematic File Version 4
+LIBS:line_sensor_color-cache
 EELAYER 29 0
 EELAYER END
@@
 F 0 "U2" H 2317 7397 60  0000 C CNN
 F 1 "XH_2" H 2317 7291 60  0000 C CNN
-F 2 "" H 2350 7100 60  0000 C CNN
+F 2 "" H 2350 7100 60  0001 C CNN
 F 3 "" H 2350 7100 60  0000 C CNN
 	1    2350 7100
@@
 F 0 "U3" H 3017 7397 60  0000 C CNN
 F 1 "XH_2" H 3017 7291 60  0000 C CNN
-F 2 "" H 3050 7100 60  0000 C CNN
+F 2 "" H 3050 7100 60  0001 C CNN
 F 3 "" H 3050 7100 60  0000 C CNN
 	1    3050 7100
@@
 F 0 "U1" H 2317 6797 60  0000 C CNN
 F 1 "XH_2" H 2317 6691 60  0000 C CNN
-F 2 "" H 2350 6500 60  0000 C CNN
+F 2 "" H 2350 6500 60  0001 C CNN
 F 3 "" H 2350 6500 60  0000 C CNN
 	1    2350 6500
@@
 F 0 "U4" H 7800 4947 60  0000 C CNN
 F 1 "NJM7800SDL1" H 7800 4841 60  0000 C CNN
-F 2 "" H 7800 4600 60  0000 C CNN
+F 2 "" H 7800 4600 60  0001 C CNN
 F 3 "" H 7800 4600 60  0000 C CNN
 	1    7800 4600
@@
 F 0 "A1" H 4158 7815 50  0000 C CNN
 F 1 "NUCLEO-F303K8" H 4158 7724 50  0000 C CNN
-F 2 "MODULE_NUCLEO-F303K8" H 4050 6850 50  0001 L BNN
+F 2 "MyFootprint:NUCLEO_F303K8" H 4050 6850 50  0001 L BNN
 F 3 "" H 4050 6850 50  0001 L BNN
 F 4 "Unavailable" H 4050 6850 50  0001 L BNN "フィールド4"
@@
 F 0 "A1" H 5708 7815 50  0000 C CNN
 F 1 "NUCLEO-F303K8" H 5708 7724 50  0000 C CNN
-F 2 "MODULE_NUCLEO-F303K8" H 5600 6850 50  0001 L BNN
+F 2 "MyFootprint:NUCLEO_F303K8" H 5600 6850 50  0001 L BNN
 F 3 "" H 5600 6850 50  0001 L BNN
 F 4 "Unavailable" H 5600 6850 50  0001 L BNN "フィールド4"

Commit message: update: ライブラリの更新
Parts:
- removed U1, U2, U3: XH_2, symbol MyComponent:XH_2
- removed U4: NJM7800SDL1, symbol MyComponent:NJM7800SDL1
- added J1, J2, J3: Conn_01x02_Male, Connector_JST:JST_XH_S2B-XH-A_1x02_P2.50mm_Horizontal, symbol Connector:Conn_01x02_Male
- added U1: NJM7805SDL1-MyComponent, Package_TO_SOT_SMD:TO-252-3_TabPin2, symbol line_sensor_color-rescue:NJM7805SDL1-MyComponent
- A1: symbol MyComponent:NUCLEO-F303K8 -> line_sensor_color-rescue:NUCLEO-F303K8-MyComponent
- R1, R10, R11, R12, R13, R14, R15, R16, R2, R24, R3, R4, R5, R6, R7, R8, R9: footprint Resistor_THT:R_Axial_DIN0204_L3.6mm_D1.6mm_P7.62mm_Horizontal -> Resistor_THT:R_Axial_DIN0207_L6.3mm_D2.5mm_P7.62mm_Horizontal
- S1, S2, S3, S4, S5, S6, S7: footprint (none) -> MyFootprint:S9032-02; symbol MyComponent:S9032-02 -> line_sensor_color-rescue:S9032-02-MyComponent
- SW1, SW2, SW3, SW4, SW5, SW6: footprint Package_DIP:DIP-6_W7.62mm -> Button_Switch_THT:SW_DIP_SPSTx03_Slide_6.7x9.18mm_W7.62mm_P2.54mm_LowProfile
Connections:
- net +5V: now also J2.1 (Pin_1), U1.3 (Vo)
- net +BATT: now also J3.1 (Pin_1), U1.1 (Vi)
- net CAN_H: now also J1.1 (Pin_1)
- net CAN_L: now also J1.2 (Pin_2)
- net GND: now also J2.2 (Pin_2), J3.2 (Pin_2), U1.2 (GND)
